File: boards/logic/logic.kicad_pcb (KiCad board)
At the start: 2 copper layers, 48.3 x 57.8 mm, 45 parts, among them IC1 ATTINY85-S, P1 5V_IN, P2 PROG_CONN, P3 DSPLY_CONN, Q1 Q_NPN_EBC, Q2 Q_NPN_EBC, Q3 Q_NPN_EBC, Q4 Q_NPN_EBC, Q5 Q_NPN_EBC, Q6 Q_NPN_EBC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

Commit message: Add final silk screen.
Parts:
- moved G*** 5.90 mm to (137.5, 120.5)
- moved G*** 0.94 mm to (137.4, 117.0)
Other:
- board text added: "A1"
Changed lines of the file:
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@@
 (kicad_pcb (version 4) (host pcbnew 4.0.2-stable)
   (general
-    (links 0)
+    (links 117)
     (no_connects 0)
     (area 121.209999 88.824999 169.620001 146.760001)
     (thickness 1.6)
-    (drawings 29)
+    (drawings 30)
     (tracks 569)
     (zones 0)
@@
   )
   (module te_logos:te_22mm_width (layer B.Cu)
-    (at 137.7188 117.856 180)
+    (at 137.414 116.967 180)
     (fp_text reference G*** (at 0 0 180) (layer B.SilkS) hide
       (effects (font (thickness 0.3)) (justify mirror))
@@
   )
   (module te_logos:te_text_22mm_width (layer B.Cu)
-    (at 137.3124 114.5794 180)
+    (at 137.5156 120.4722 180)
     (fp_text reference G*** (at 0 0 180) (layer B.SilkS) hide
       (effects (font (thickness 0.3)) (justify mirror))
@@
       (xy 8.297753 0.632539)) (layer B.SilkS) (width 0.01))
   )
+  (gr_text A1 (at 123.317 90.9574) (layer F.SilkS)
+    (effects (font (size 1 1) (thickness 0.2)))
+  )
   (gr_circle (center 166.37 130.81) (end 170.434 130.81) (layer F.Fab) (width 0.15))
